File: PCB/AlterErgo.sch (KiCad schematic (older format))
At the start: 94 parts, among them J1 GS3, J2 SJ-43514, J3 GS3, SW0:10 SW_Push, SW0:11 SW_Push, SW0:12 SW_Push, SW0:7 SW_Push, SW0:8 SW_Push, SW0:9 SW_Push, SW1 SW_SPST, SW1:10 SW_Push, SW1:11 SW_Push, SW1:12 SW_Push, SW1:13 SW_Push, SW1:7 SW_Push, SW1:8 SW_Push, SW1:9 SW_Push, SW2:10 SW_Push, SW2:11 SW_Push, SW2:12 SW_Push, SW2:13 SW_Push, SW2:7 SW_Push, SW2:8 SW_Push, SW2:9 SW_Push, SW3:10 SW_Push, SW3:11 SW_Push, SW3:12 SW_Push, SW3:13 SW_Push, SW3:8 SW_Push, SW3:9 SW_Push, SW4:10 SW_Push, SW4:11 SW_Push, SW4:12 SW_Push, SW4:13 SW_Push, SW4:7 SW_Push, SW4:8 SW_Push, SW4:9 SW_Push, SW5:10 SW_Push, SW5:11 SW_Push, SW5:12 SW_Push, SW5:13 SW_Push, SW5:7 SW_Push, SW5:8 SW_Push, SW5:9 SW_Push, U1 Feather32u4Bluefruit, U2 MCP23018

Commit message: Update main PCB schematic to use breakout board footprint in place of controller/IO Expander and TRRS jack
Parts:
- removed J1, J3: GS3, Connectors:GS3, symbol GS3
- removed J2: SJ-43514, keyboard_accessories:TRRS_Jack_SJ-43514_reversible, symbol SJ-43514
- removed R1, R2: 2.2k, Resistors_THT:R_Axial_DIN0207_L6.3mm_D2.5mm_P7.62mm_Horizontal, symbol R
- removed U2: MCP23018, Housings_DIP:DIP-28_W7.62mm, symbol MCP23018
- added SW2: SW_Push, Buttons_Switches_THT:SW_PUSH_6mm, symbol SW_Push
- added U2: FeatherBreakout, IOBreakout:FeatherBreakout, symbol FeatherBreakout
- U1: value Feather32u4Bluefruit -> FeatherBreakout; footprint keyboard_accessories:Feather32u4Bluefruit -> IOBreakout:FeatherBreakout; symbol Feather32u4Bluefruit -> FeatherBreakout
Connections:
- net +3V3: now also U2.27 (+3V3)
- net GND: now also SW2.2, U2.25 (GND)
- net SCL: now also U2.11 (GPIO_3)
- net SDA: now also U2.12 (GPIO_2)
- net ENABLE: now reaches SW1.2 (B), U1.2 (EN)
- net RESET: now reaches U1.28 (RST)
- net RESET: now also SW2.1
- net LED1: now reaches U1.4 (GPIO_13)
- net LED1: now also R3.2
- net LED2: now reaches R4.2
- net LED2: now also U1.29 (IO2)
- net LED3: now reaches R5.2
- net LED3: now also U1.30 (IO3)
- no-connect marks 8 -> 31
Other:
- note added: "Breakout for TRRS jack (for both halves)"
- note added: "Dev board in right half/IO Expander breakout in left half"
- note removed: "Dev board in right half"
- note removed: "IO expander in left half"
- note removed: "TRRS jack with jumpers to select\nwhich ring does power and which\none does ground"
- moved on the sheet: D1, D2, D3, R3, R4, R5, SW1
